File: hardware/electronics/kat_control_board/kat_control_board.kicad_sch (KiCad schematic)
At the start: 113 parts, among them J1 USB_C_Receptacle_USB2.0, J10 Conn_01x04, J11 Conn_01x04, J12 Conn_01x04, J13 Conn_01x04, J14 Conn_01x04, J15 Conn_01x04, J16 Conn_01x04, J17 Conn_01x02, J18 Conn_01x04, J19 Conn_01x04, J2 Conn_01x04, J20 Conn_01x02, J21 Conn_01x02, J22 Conn_01x02, J23 Conn_01x02, J24 Conn_01x02, J25 Conn_01x02, J26 Conn_01x02, J27 Conn_01x02, J3 Conn_01x04, J4 Conn_01x04, J5 Conn_01x04, J6 Conn_01x04, J7 Conn_01x04, J8 Conn_01x04, J9 Conn_01x04, Q1 AO3400A, Q2 AO3400A, Q3 AO3400A, Q4 AO3400A, Q5 AO3400A, SW1 SW_SPST, SW2 SW_SPST, U1 RP2040, U2 W25Q128JVS, U3 SN74HC4851, U4 74HCT244, U5 74HCT244, U6 SIC431, U7 XC6206PxxxMR, Y1 12MHz

Commit message: Added rev1 PCB design
Parts:
- added H1, H2, H3: MountingHole, MountingHole:MountingHole_3.5mm_Pad_Via, symbol Mechanical:MountingHole
- added J28: Conn_01x04, M_Connectors:DB2ERC-3.5-4P, symbol Connector_Generic:Conn_01x04
- added J29, J30, J31, J32: Conn_02x30_Odd_Even, Connector_PinHeader_2.54mm:PinHeader_2x30_P2.54mm_Vertical, symbol Connector_Generic:Conn_02x30_Odd_Even
- added LOGO1: Logo_Open_Hardware_Small, M_LOGOS:kinki_yokai_logo, symbol Graphic:Logo_Open_Hardware_Small
- R1, R2: value 27R4 -> 27R; footprint Resistor_SMD:R_0402_1005Metric -> Resistor_SMD:R_0603_1608Metric; JLC C274349 -> C25190
Connections:
- net +12V: now also J28.1 (Pin_1), J28.2 (Pin_2), J32.10 (Pin_10), J32.12 (Pin_12), J32.2 (Pin_2), J32.4 (Pin_4), J32.6 (Pin_6), J32.8 (Pin_8)
- net +5V: now also J29.1 (Pin_1), J29.2 (Pin_2), J30.1 (Pin_1), J30.2 (Pin_2), J31.1 (Pin_1), J31.2 (Pin_2)
- net GND: now also J28.3 (Pin_3), J28.4 (Pin_4), J29.57 (Pin_57), J29.58 (Pin_58), J29.59 (Pin_59), J29.60 (Pin_60), J30.57 (Pin_57), J30.58 (Pin_58), J30.59 (Pin_59), J30.60 (Pin_60), J31.57 (Pin_57), J31.58 (Pin_58), J31.59 (Pin_59), J31.60 (Pin_60), J32.57 (Pin_57), J32.58 (Pin_58), J32.59 (Pin_59), J32.60 (Pin_60)
- net AMUX_A: now reaches U1.35 (GPIO23), U3.11 (A)
- net AMUX_B: now reaches U1.36 (GPIO24), U3.10 (B)
- net AMUX_C: now reaches U1.37 (GPIO25), U3.9 (C)
- net AMUX_X: now reaches U1.38 (GPIO26_ADC0), U3.3 (X)
Other:
- note added: "EXPANSION"
- note added: "LED PORTS"
- note added: "MECHANICAL"
- note added: "POWER_IN, 5V SMPS, 3V3 LDO"
- note added: "PULL SENSORS"
- note added: "RP2040"
- note added: "RP2040 FLASH"
- note added: "SWITCHED 12V, 12V OUT"
- note added: "USB"
- moved on the sheet: C1, C10, C11, C12, C13, C14, C15, C16, C17, C18, C19, C2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
